File: rak3172LP-SIP/rak3172sip.kicad_pcb (KiCad board)
At the start: 2 copper layers, 46.5 x 29 mm, 46 parts, among them J1 U.FL, J2 Conn_ARM_SWD_TagConnect_TC203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, J4 Conn_01x03_Socket, J5 Conn_01x02_Socket, J6 Conn_01x08_Socket, U1 RAK3172-SIP

Commit message: HW V0.04
Parts:
- removed L3: Bead120, Inductor_SMD:L_0402_1005Metric
- Z1: value 0 -> 8.2nH
- Z3: value tbd -> 5.6nH
- Z4: value tbd -> np
Connections:
- C11 pad 1: Net-(U1-VDDPA) -> VPA
- C14 pad 1: Net-(U1-VFBSMPS) -> VPA
- C15 pad 1: Net-(U1-VFBSMPS) -> VPA
- L2 pad 1: Net-(U1-VFBSMPS) -> VPA
- U1 pad 10: Net-(U1-VFBSMPS) -> VPA
- U1 pad 53: Net-(U1-VDDPA) -> VPA
Routing:
- net VPA: track 0.00 -> 25.1 mm, vias 0 -> 2
- net Net-(U1-VDDPA): track 8.38 -> 0.00 mm
- net Net-(U1-VFBSMPS): track 7.39 -> 0.00 mm
- net +3V3: track 109.0 -> 108.0 mm
- net GND: track 135.7 -> 134.9 mm, vias 61 -> 62
