File: rak3172LP-SIP/rak3172sip.kicad_sch (KiCad schematic)
At the start: 42 parts, among them J1 U.FL, J2 Conn_ARM_SWD_TagConnect_TC203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, J4 Conn_01x03_Socket, J5 Conn_01x02_Socket, J6 Conn_01x08_Socket, U1 RAK3172-SIP

Commit message: 0v02
Parts:
- J1, TP3: now left out of the parts list
Changed lines of the file:
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@@
 	(title_block
 		(title "RAK3172(LP)-SIP")
-		(date "2025-06-13")
-		(rev "V0.01")
+		(date "2025-06-16")
+		(rev "V0.02")
 		(company "JoEmbedded.de")
 	)
@@
 		(unit 1)
 		(exclude_from_sim no)
-		(in_bom yes)
+		(in_bom no)
 		(on_board yes)
 		(dnp no)
@@
 			)
 		)
-		(property "Datasheet" ""
+		(property "Datasheet" "https://store.rakwireless.com/products/wisduo-module-rak3172-sip?variant=42482784796870"
 			(at 143.51 88.9 0)
 			(effects
@@
 			)
 		)
-		(property "Description" ""
+		(property "Description" "RAK3172LP-SiP / 8XXMHz for EU868/IN865/RU864  SKU: 305049"
 			(at 143.51 88.9 0)
 			(effects
@@
 		(unit 1)
 		(exclude_from_sim no)
-		(in_bom yes)
+		(in_bom no)
 		(on_board yes)
 		(dnp no)

Commit message: Rak3172LP V0.03
Parts:
- Z1: value 0 -> 8.2nH; now fitted
- Z2: now fitted
- Z3: value tbd -> 5.6nH; now fitted
- Z4: value tbd -> np
Other:
- note added: "Variants: J1: Assembled for external Antenna Z2: Assembled for internal Antenna Z1: dto Z3: dto Z1,Z3: depending on PCB material"
- note removed: "Z1: adjusts ANT to el. Lambda/4 Z2-4: tbd. for Impedance matching"
Changed lines of the file:
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@@
 	(title_block
 		(title "RAK3172(LP)-SIP")
-		(date "2025-06-16")
-		(rev "V0.02")
+		(date "2025-07-18")
+		(rev "V0.03")
 		(company "JoEmbedded.de")
 	)
@@
 		)
 	)
-	(text "Z1: adjusts ANT to el. Lambda/4\nZ2-4: tbd. for Impedance matching"
+	(text "Variants:\nJ1: Assembled for external Antenna\n\nZ2: Assembled for internal Antenna\nZ1: dto\nZ3: dto\n\nZ1,Z3: depending on PCB material\n"
 		(exclude_from_sim no)
-		(at 245.364 105.918 0)
+		(at 244.602 117.602 0)
 		(effects
 			(font
@@
 		)
 	)
+	(polyline
+		(pts
+			(xy 237.49 105.41) (xy 237.49 110.49)
+		)
+		(stroke
+			(width 0)
+			(type default)
+		)
+	)
 	(wire
 		(pts
@@
 		)
 	)
+	(polyline
+		(pts
+			(xy 236.855 106.68) (xy 237.49 105.41)
+		)
+		(stroke
+			(width 0)
+			(type default)
+		)
+	)
 	(wire
 		(pts
@@
 		)
 	)
+	(polyline
+		(pts
+			(xy 254.635 92.71) (xy 255.27 91.44)
+		)
+		(stroke
+			(width 0)
+			(type default)
+		)
+	)
 	(wire
 		(pts
@@
 		)
 	)
+	(polyline
+		(pts
+			(xy 255.27 91.44) (xy 255.27 110.49)
+		)
+		(stroke
+			(width 0)
+			(type default)
+		)
+	)
 	(wire
 		(pts
@@
 		)
 	)
+	(polyline
+		(pts
+			(xy 254 110.49) (xy 255.27 110.49)
+		)
+		(stroke
+			(width 0)
+			(type default)
+		)
+	)
 	(wire
 		(pts
@@
 		)
 	)
+	(polyline
+		(pts
+			(xy 243.84 110.49) (xy 237.49 110.49)
+		)
+		(stroke
+			(width 0)
+			(type default)
+		)
+	)
 	(wire
 		(pts
@@
 		)
 	)
+	(polyline
+		(pts
+			(xy 255.905 92.71) (xy 255.27 91.44)
+		)
+		(stroke
+			(width 0)
+			(type default)
+		)
+	)
 	(wire
 		(pts
@@
 		)
 	)
+	(polyline
+		(pts
+			(xy 238.125 106.68) (xy 237.49 105.41)
+		)
+		(stroke
+			(width 0)
+			(type default)
+		)
+	)
 	(global_label "SDA2"
 		(shape input)
@@
 			)
 		)
-		(property "Value" "tbd"
+		(property "Value" "np"
 			(at 250.19 93.9862 0)
 			(effects
@@
 		(in_bom yes)
 		(on_board yes)
-		(dnp yes)
+		(dnp no)
 		(fields_autoplaced yes)
 		(property "Reference" "Z2"
@@
 		(in_bom yes)
 		(on_board yes)
-		(dnp yes)
+		(dnp no)
 		(fields_autoplaced yes)
 		(property "Reference" "Z1"
@@
 			)
 		)
-		(property "Value" "0"
+		(property "Value" "8.2nH"
 			(at 273.05 86.36 90)
 			(effects
@@
 		(in_bom yes)
 		(on_board yes)
-		(dnp yes)
+		(dnp no)
 		(fields_autoplaced yes)
 		(property "Reference" "Z3"
@@
 			)
 		)
-		(property "Value" "tbd"
+		(property "Value" "5.6nH"
 			(at 265.43 93.9862 0)
 			(effects

Commit message: HW V0.04
Parts:
- removed L3: Bead120, Inductor_SMD:L_0402_1005Metric, symbol Device:L_Ferrite_Small
Connections:
- net VPA: now reaches C14.1, C15.1, L2.1, U1.10 (VFBSMPS)
- net VPA: now also C11.1, U1.53 (VDDPA)
Other:
- note added: "LowPower-Version!"
- moved on the sheet: ANT1

Commit message: 0.04
Other:
- note added: "RAK3172LP, ST50HE (Modules technically identical)"
Changed lines of the file:
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@@
+		)
+	)
+	(text "RAK3172LP, ST50HE\n(Modules technically identical)\n"
+		(exclude_from_sim no)
+		(at 140.97 43.688 0)
+		(effects
+			(font
+				(size 1.27 1.27)
+			)
 		)
 	)

Commit message: V1.8
Other:
- note added: "*todo* - RESET auf PIN führen (fuer Verw. als Modem)"
Changed lines of the file:
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@@
+		)
+	)
+	(text "*todo*\n- RESET auf PIN führen (fuer Verw. als Modem)"
+		(exclude_from_sim no)
+		(at 35.306 168.402 0)
+		(effects
+			(font
+				(size 2.54 2.54)
+			)
+			(justify left)
 		)
 	)
